File: pico_expansion_board/pico_expansion_board.kicad_pcb (KiCad board)
At the start: 4 copper layers, 99.1 x 69.8 mm, 51 parts, among them IC1 TPS5450DDA, J1 DC12V/24V, J10 CAN_L, J2 TMC2209 Motor 1, J3 TMC2209 Motor 2, J4 Motor 1, J5 Motor 2, J6 Straight Through, J7 NULL Modem, J8 EXP1, J9 EXP2, SW1 SW_Push, U1 MAX232, U2 MCP2542FDxMF, U3 Pico, U5 CAT24C256

Commit message: Update production file, update STEP models
Parts:
- moved TP8 6.86 mm to (75.7, 63.8)
- moved TP7 5.59 mm to (69.3, 63.8)
- moved C4 0.84 mm to (122.4, 81.8)
Connections:
- U3 pad 1: SCALE_UART_RX -> SCALE_UART_TX
- U3 pad 2: SCALE_UART_TX -> SCALE_UART_RX
Routing:
- net SCALE_UART_RX: track 72.9 -> 65.5 mm, vias 2 -> 1
- net SCALE_UART_TX: track 67.4 -> 74.1 mm
- net +5V: track 48.7 -> 51.2 mm
- net BTN_EN1: track 29.7 -> 31.9 mm
- net LCD_RST: track 37.9 -> 40.1 mm
- net BTN_EN2: track 25.6 -> 27.7 mm
- net LCD_CS: track 33.0 -> 34.8 mm
- net GND: track 64.3 -> 65.5 mm
- net LED_SCK: track 39.8 -> 41.0 mm
- net LCD_MOSI: track 39.1 -> 40.2 mm
- net Net-(J10-Pin_2): track 38.3 -> 39.0 mm
Other:
- outline, holes or cut-outs redrawn

Commit message: Update to v0.2, include additional caps for StepStick driver VM input
Parts:
- added C11: 100uF, Capacitor_SMD:CP_Elec_6.3x7.7, F.Cu at (69.6, 104.9)
- added C12: 100uF, Capacitor_SMD:CP_Elec_6.3x7.7, F.Cu at (69.6, 78.8)
- moved JP4 8.38 mm to (70.1, 97.5)
- moved JP2 7.12 mm to (70.0, 71.6)
- moved JP3 7.12 mm to (68.1, 94.2)
- moved JP1 5.92 mm to (67.9, 68.3)
- moved TP7 1.02 mm to (69.3, 62.7)
- moved TP4 0.25 mm to (68.1, 88.9)
Routing:
- net VCC: track 23.3 -> 45.4 mm, vias 1 -> 3
- net GND: track 65.5 -> 85.2 mm
- net Net-(J3-PDN): track 5.80 -> 9.02 mm
- net Net-(J2-PDN): track 5.97 -> 9.09 mm
- net MOTOR_UART: track 58.3 -> 55.8 mm, vias 2 -> 3
- net Net-(J2-UART): track 6.16 -> 8.38 mm
- net Net-(J3-UART): track 6.65 -> 8.28 mm
Other:
- board text added: "EN"
- board text added: "OpenTricker Controller v0.2"
- board text added: "VM"
- board text removed: "OpenTricker Controller v0.1"
